Commit message: fix pitch

File: resources/models/gimbal_snippets.xacro (robot description, xacro)
@@ -29,5 +29,5 @@
             <parent link="${link_name}"/>
             <child link="${child_link}"/>
-            <axis xyz="1 0 0"/>
+            <axis xyz="0 1 0"/>
             <dynamics damping="0"/>
             <dynamics friction="1000"/>
@@ -107,5 +107,5 @@
     </xacro:macro>
     <xacro:macro name="bottom_1D_gimbal" params="namespace parent_link *origin visible">
-        <gimbal_base_joint  joint_name="${namespace}/pitch_joint" link_name="${namespace}/gimbal_base_link" child_link="${namespace}/camera_mount_link" visible="${visible}" rpy="0 0 ${pi/2}" parent_link="${parent_link}">
+        <gimbal_base_joint  joint_name="${namespace}/pitch_joint" link_name="${namespace}/gimbal_base_link" child_link="${namespace}/camera_mount_link" visible="${visible}" rpy="0 0 0" parent_link="${parent_link}">
             <xacro:insert_block name="origin" />
         </gimbal_base_joint>
@@ -115,5 +115,5 @@
                 <origin xyz="0 0 0"/>
                 <geometry>
-                    <box size="0.1 0.05 0.01" />
+                    <box size="0.05 0.1 0.01" />
                 </geometry>
             </visual>

Commit message: add 2D gimbal
for simplicity only small use of xacro

File: resources/models/gimbal_snippets.xacro (robot description, xacro)
@@ -137,3 +137,91 @@
         </gazebo>
     </xacro:macro>
+    <xacro:macro name="bottom_2D_gimbal" params="namespace parent_link *origin visible">
+        <joint name="gimbal_fix" type="prismatic"> <!-- prismatic joint with zero limits(default) is a hack for a fixed joint (needed on gazebo7)-->
+            <parent link="${parent_link}"/>
+            <child link="${namespace}/gimbal_base_link"/>
+            <axis xyz="1 0 0"/>
+            <dynamics damping="0"/>
+            <dynamics friction="100"/>
+            <limit velocity="1e+16" effort="1e+16" />
+            <xacro:insert_block name="origin" />
+        </joint>
+        <link name='${namespace}/gimbal_base_link'>
+            <xacro:if value="${visible}">
+                <visual>
+                    <origin xyz="0 0 0"/>
+                    <geometry>
+                        <box size="0.01 0.01 0.04" />
+                    </geometry>
+                </visual>
+            </xacro:if>
+            <inertial>
+                <mass value="1e-5" />
+                <origin xyz="0 0 0" rpy="0 0 0" />
+                <inertia ixx="1e-6" ixy="0" ixz="0" iyy="1e-6" iyz="0" izz="1e-6" />
+            </inertial>
+        </link>
+        <joint name="${namespace}/pitch_joint" type="continuous">
+            <parent link="${namespace}/gimbal_base_link"/>
+            <child link="${namespace}/inter_link"/>
+            <axis xyz="0 1 0"/>
+            <dynamics damping="0"/>
+            <dynamics friction="1000"/>
+            <limit velocity="1e+16" effort="1e+16" />
+            <origin xyz="0 0 0" rpy="0.0 0.0 0.0"/>
+        </joint>
+        <link name='${namespace}/inter_link'>
+            <xacro:if value="${visible}">
+                <visual>
+                    <origin xyz="0 0 0"/>
+                    <geometry>
+                        <box size="0.01 0.01 0.01" />
+                    </geometry>
+                </visual>
+            </xacro:if>
+            <inertial>
+                <mass value="1e-5" />
+                <origin xyz="0 0 0" rpy="0 0 0" />
+                <inertia ixx="1e-6" ixy="0" ixz="0" iyy="1e-6" iyz="0" izz="1e-6" />
+            </inertial>
+        </link>
+        <joint name="${namespace}/yaw_joint" type="continuous">
+            <parent link="${namespace}/inter_link"/>
+            <child link="${namespace}/camera_mount_link"/>
+            <axis xyz="0 0 1"/>
+            <dynamics damping="0"/>
+            <dynamics friction="1000"/>
+            <limit velocity="1e+16" effort="1e+16" />
+            <origin xyz="0 0 0" rpy="0.0 0.0 0.0"/>
+        </joint>
+        <link name='${namespace}/camera_mount_link'>
+            <xacro:if value="${visible}">
+                <visual >
+                    <origin xyz="0 0 0"/>
+                    <geometry>
+                        <box size="0.02 0.06 0.04" />
+                    </geometry>
+                </visual>
+            </xacro:if>
+            <inertial>
+                <mass value="1e-5" />
+                <origin xyz="0 0 0" rpy="0 0 0" />
+                <inertia ixx="1e-6" ixy="0" ixz="0" iyy="1e-6" iyz="0" izz="1e-6" />
+            </inertial>
+        </link>
+        <gazebo >
+            <plugin name="gimbal_controller" filename="libgazebo_poltergeist_gimbal_plugin.so">
+                <robot_namespace>/${namespace}</robot_namespace>
+                <pitch_joint_name>${namespace}/pitch_joint</pitch_joint_name>
+                <pitch_direction>1</pitch_direction>
+                <pitch_zero>0</pitch_zero>
+                <yaw_joint_name>${namespace}/yaw_joint</yaw_joint_name>
+                <yaw_direction>2</yaw_direction>
+                <yaw_zero>0</yaw_zero>
+                <gimbal_angular_velocity>0.5</gimbal_angular_velocity>
+                <ref_base_link>${parent_link}</ref_base_link>
+                <camera_link>${namespace}/camera_mount_link</camera_link>
+            </plugin>
+        </gazebo>
+    </xacro:macro>
 </robot>

Commit message: add setting of max_rotational_velocity from 2D gimbal

File: resources/models/gimbal_snippets.xacro (robot description, xacro)
@@ -137,5 +137,5 @@
         </gazebo>
     </xacro:macro>
-    <xacro:macro name="bottom_2D_gimbal" params="namespace parent_link *origin visible">
+    <xacro:macro name="bottom_2D_gimbal" params="namespace parent_link *origin visible max_rotational_velocity">
         <joint name="gimbal_fix" type="prismatic"> <!-- prismatic joint with zero limits(default) is a hack for a fixed joint (needed on gazebo7)-->
             <parent link="${parent_link}"/>
@@ -219,5 +219,5 @@
                 <yaw_direction>2</yaw_direction>
                 <yaw_zero>0</yaw_zero>
-                <gimbal_angular_velocity>0.5</gimbal_angular_velocity>
+                <gimbal_angular_velocity>${max_rotational_velocity}</gimbal_angular_velocity>
                 <ref_base_link>${parent_link}</ref_base_link>
                 <camera_link>${namespace}/camera_mount_link</camera_link>
